Commit message: 修复一些问题,导致运行不起来

File: src/unitree_guide/unitree_ros/robots/a1_description/urdf/a1.urdf (robot description, URDF)
Before this commit: robot a1, 23 links, 22 joints
Links:
- added link laser_livox; collision mesh filename=package://a1_description/meshes/livox_mid360.dae; visual mesh filename=package://a1_description/meshes/livox_mid360.dae
- added link livox_imu_link, mass 0.001; collision box size=.001 .001 .001; visual box size=0.001 0.001 0.001
- link FL_calf: mass 0.166 -> 0.151
- link FL_hip: mass 0.696 -> 0.595
- link FL_thigh: mass 1.013 -> 0.888
- link FR_calf: mass 0.166 -> 0.151
- link FR_hip: mass 0.696 -> 0.595
- link FR_thigh: mass 1.013 -> 0.888
- link RL_calf: mass 0.166 -> 0.151
- link RL_hip: mass 0.696 -> 0.595
- link RL_thigh: mass 1.013 -> 0.888
- link RR_calf: mass 0.166 -> 0.151
- link RR_hip: mass 0.696 -> 0.595
- link RR_thigh: mass 1.013 -> 0.888
Joints:
- added joint FL_foot_joint_get_position: type revolute, parent FL_calf, child FL_foot, origin xyz=0 0 -0.2 rpy=0 0 0, axis 0 1 0, limit lower=0 upper=0 effort=0 velocity=0
- added joint FR_foot_joint_get_position: type revolute, parent FR_calf, child FR_foot, origin xyz=0 0 -0.2 rpy=0 0 0, axis 0 1 0, limit lower=0 upper=0 effort=0 velocity=0
- added joint RL_foot_joint_get_position: type revolute, parent RL_calf, child RL_foot, origin xyz=0 0 -0.2 rpy=0 0 0, axis 0 1 0, limit lower=0 upper=0 effort=0 velocity=0
- added joint RR_foot_joint_get_position: type revolute, parent RR_calf, child RR_foot, origin xyz=0 0 -0.2 rpy=0 0 0, axis 0 1 0, limit lower=0 upper=0 effort=0 velocity=0
- added joint laser_livox_joint: type fixed, parent base, child laser_livox, origin xyz=0.2 0 0.08 rpy=0 0.785 0
- added joint livox_imu_joint: type fixed, parent laser_livox, child livox_imu_link, origin xyz=-0.011 -0.02329 0.04412 rpy=0 0 0
- joint FL_calf_joint: limit lower=-2.69653369433 upper=-0.916297857297 effort=33.5 velocity=21 -> lower=-2.6965336943312392 upper=-0.9162978572970231 effort=33.5 velocity=21
- joint FL_hip_joint: limit lower=-0.802851455917 upper=0.802851455917 effort=33.5 velocity=21 -> lower=-0.8028514559173915 upper=0.8028514559173915 effort=33.5 velocity=21
- joint FL_thigh_joint: limit lower=-1.0471975512 upper=4.18879020479 effort=33.5 velocity=21 -> lower=-1.0471975511965976 upper=4.1887902047863905 effort=33.5 velocity=21
- joint FR_calf_joint: limit lower=-2.69653369433 upper=-0.916297857297 effort=33.5 velocity=21 -> lower=-2.6965336943312392 upper=-0.9162978572970231 effort=33.5 velocity=21
- joint FR_hip_joint: limit lower=-0.802851455917 upper=0.802851455917 effort=33.5 velocity=21 -> lower=-0.8028514559173915 upper=0.8028514559173915 effort=33.5 velocity=21
- joint FR_thigh_joint: limit lower=-1.0471975512 upper=4.18879020479 effort=33.5 velocity=21 -> lower=-1.0471975511965976 upper=4.1887902047863905 effort=33.5 velocity=21
- joint RL_calf_joint: limit lower=-2.69653369433 upper=-0.916297857297 effort=33.5 velocity=21 -> lower=-2.6965336943312392 upper=-0.9162978572970231 effort=33.5 velocity=21
- joint RL_hip_joint: limit lower=-0.802851455917 upper=0.802851455917 effort=33.5 velocity=21 -> lower=-0.8028514559173915 upper=0.8028514559173915 effort=33.5 velocity=21
- joint RL_thigh_joint: limit lower=-1.0471975512 upper=4.18879020479 effort=33.5 velocity=21 -> lower=-1.0471975511965976 upper=4.1887902047863905 effort=33.5 velocity=21
- joint RR_calf_joint: limit lower=-2.69653369433 upper=-0.916297857297 effort=33.5 velocity=21 -> lower=-2.6965336943312392 upper=-0.9162978572970231 effort=33.5 velocity=21
- joint RR_hip_joint: limit lower=-0.802851455917 upper=0.802851455917 effort=33.5 velocity=21 -> lower=-0.8028514559173915 upper=0.8028514559173915 effort=33.5 velocity=21
- joint RR_thigh_joint: limit lower=-1.0471975512 upper=4.18879020479 effort=33.5 velocity=21 -> lower=-1.0471975511965976 upper=4.1887902047863905 effort=33.5 velocity=21

File: src/unitree_guide/unitree_ros/robots/a1_description/xacro/gazebo.xacro (robot description, xacro)
@@ -8,5 +8,5 @@
             </ros>
             <robot_param>robot_description</robot_param>
-            <robot_param_node>robot_state_publisher</robot_param_node>
+            <robot_param_node>/robot_state_publisher</robot_param_node>
             <parameters>$(find a1_description)/config/robot_control.yaml</parameters>
         </plugin>

File: src/unitree_guide/unitree_ros/robots/a1_description/xacro/leg.xacro (robot description, xacro)
@@ -1,5 +1,4 @@
 <?xml version="1.0"?>
 <robot xmlns:xacro="http://www.ros.org/wiki/xacro">
-    <xacro:include filename="$(find a1_description)/xacro/transmission.xacro"/>
     <xacro:macro name="leg" params="name mirror mirror_dae front_hind front_hind_dae *origin">
         <joint name="${name}_hip_joint" type="revolute">

File: src/unitree_guide/unitree_ros/robots/a1_description/xacro/robot.xacro (robot description, xacro)
@@ -7,4 +7,5 @@
     <xacro:include filename="$(find a1_description)/xacro/stairs.xacro"/>
     <xacro:include filename="$(find a1_description)/xacro/gazebo.xacro"/>
+    <xacro:include filename="$(find a1_description)/xacro/transmission.xacro"/>
     <!-- <xacro:include filename="$(find a1_gazebo)/launch/stairs.urdf.xacro"/> -->
     <!-- <xacro:stairs stairs="15" xpos="0" ypos="0" zpos="0" /> -->
