Commit message: 修复控制以及gazebo这些bug

File: src/unitree_guide/unitree_ros/robots/a1_description/xacro/gazebo.xacro (robot description, xacro)
@@ -7,6 +7,4 @@
                 <namespace>/a1_gazebo</namespace>
             </ros>
-            <robot_param>robot_description</robot_param>
-            <robot_param_node>/robot_state_publisher</robot_param_node>
             <parameters>$(find a1_description)/config/robot_control.yaml</parameters>
         </plugin>
@@ -40,5 +38,5 @@
                 <remapping>wrench:=/apply_force/trunk</remapping>
             </ros>
-            <link_name>trunk</link_name>
+            <link_name>base</link_name>
         </plugin>
     </gazebo>
@@ -69,5 +67,5 @@
             <update_rate>100</update_rate>
             <body_name>base</body_name>
-            <frame_name>trunk</frame_name>
+            <frame_name>base</frame_name>
             <xyz_offset>0 0 0</xyz_offset>
             <rpy_offset>0 0 0</rpy_offset>
@@ -145,5 +143,5 @@
         <sensor name="FR_foot_contact" type="contact">
         <update_rate>100</update_rate>
-        <plugin name="contactPlugin" filename="libunitreeFootContactPlugin.so"/>
+        <plugin name="FR_contactPlugin" filename="libunitreeFootContactPlugin.so"/>
         <contact>
             <collision>FR_calf_fixed_joint_lump__FR_foot_collision_1</collision>
@@ -154,5 +152,5 @@
         <sensor name="FL_foot_contact" type="contact">
         <update_rate>100</update_rate>
-        <plugin name="contactPlugin" filename="libunitreeFootContactPlugin.so"/>
+        <plugin name="FL_contactPlugin" filename="libunitreeFootContactPlugin.so"/>
         <contact>
             <collision>FL_calf_fixed_joint_lump__FL_foot_collision_1</collision>
@@ -163,5 +161,5 @@
         <sensor name="RR_foot_contact" type="contact">
         <update_rate>100</update_rate>
-        <plugin name="contactPlugin" filename="libunitreeFootContactPlugin.so"/>
+        <plugin name="RR_contactPlugin" filename="libunitreeFootContactPlugin.so"/>
         <contact>
             <collision>RR_calf_fixed_joint_lump__RR_foot_collision_1</collision>
@@ -172,5 +170,5 @@
         <sensor name="RL_foot_contact" type="contact">
         <update_rate>100</update_rate>
-        <plugin name="contactPlugin" filename="libunitreeFootContactPlugin.so"/>
+        <plugin name="RL_contactPlugin" filename="libunitreeFootContactPlugin.so"/>
         <contact>
             <collision>RL_calf_fixed_joint_lump__RL_foot_collision_1</collision>
@@ -181,5 +179,5 @@
     <gazebo reference="FR_foot">
         <visual>
-            <plugin name="drawForcePlugin" filename="libunitreeDrawForcePlugin.so">
+            <plugin name="FR_drawForcePlugin" filename="libunitreeDrawForcePlugin.so">
                 <topicName>FR_foot_contact</topicName>
             </plugin>
@@ -188,5 +186,5 @@
     <gazebo reference="FL_foot">
         <visual>
-            <plugin name="drawForcePlugin" filename="libunitreeDrawForcePlugin.so">
+            <plugin name="FL_drawForcePlugin" filename="libunitreeDrawForcePlugin.so">
                 <topicName>FL_foot_contact</topicName>
             </plugin>
@@ -195,5 +193,5 @@
     <gazebo reference="RR_foot">
         <visual>
-            <plugin name="drawForcePlugin" filename="libunitreeDrawForcePlugin.so">
+            <plugin name="RR_drawForcePlugin" filename="libunitreeDrawForcePlugin.so">
                 <topicName>RR_foot_contact</topicName>
             </plugin>
@@ -202,5 +200,5 @@
     <gazebo reference="RL_foot">
         <visual>
-            <plugin name="drawForcePlugin" filename="libunitreeDrawForcePlugin.so">
+            <plugin name="RL_drawForcePlugin" filename="libunitreeDrawForcePlugin.so">
                 <topicName>RL_foot_contact</topicName>
             </plugin>
@@ -372,5 +370,5 @@
                     <samples>24000</samples>
                     <downsample>1</downsample>
-                    <csv_file_name>package://a1_description/scan_mode/mid360.csv</csv_file_name>
+                    <csv_file_name>$(find a1_description)/scan_mode/mid360.csv</csv_file_name>
                     <ros_topic>/scan</ros_topic>
                     <frameName>laser_livox</frameName>
@@ -381,9 +379,9 @@
     <gazebo reference="livox_imu_link">
     <gravity>true</gravity>
-    <sensor name="imu_sensor" type="imu">
+    <sensor name="livox_imu_sensor" type="imu">
         <always_on>true</always_on>
         <update_rate>1000</update_rate>
         <visualize>true</visualize>
-        <plugin filename="libgazebo_ros_imu_sensor.so" name="imu_plugin">
+        <plugin filename="libgazebo_ros_imu_sensor.so" name="livox_imu_plugin">
             <ros>
                 <namespace>/a1_gazebo</namespace>

File: src/unitree_guide/unitree_ros/robots/a1_description/xacro/leg.xacro (robot description, xacro)
@@ -130,9 +130,4 @@
             </inertial>
         </link>
-        <joint name="${name}_foot_fixed" type="fixed">
-            <origin rpy="0 0 0" xyz="0 0 ${-(calf_length)}"/>
-            <parent link="${name}_calf"/>
-            <child link="${name}_foot"/>
-        </joint>
         <joint name="${name}_foot_joint_get_position" type="revolute">
             <origin rpy="0 0 0" xyz="0 0 ${-(calf_length)}"/>
